Commit message: warning of inertia fixed

File: ws_moveit/src/arm_assembly_4/urdf/arm_assembly_4.urdf (robot description, URDF)
Before this commit: robot arm_assembly_4, 7 links, 6 joints
Links:
- added link dummy_link
Joints:
- added joint dummy_joint: type fixed, parent dummy_link, child base_link
