Commit message: assembly_6 updated

File: ws_moveit/src/arm_assembly_6/urdf/arm_assembly_6.urdf (robot description, URDF)
Before this commit: robot arm_assembly_6, 7 links, 6 joints
Joints:
- joint joint2: origin xyz=-0.00052573 0.032998 0.027656 rpy=1.5746 -1.5708 0 -> xyz=-0.00052573 0.032998 0.027656 rpy=-1.5746 -1.5708 0

Commit message: arm_assembly_6_moveit_config added, working

File: ws_moveit/src/arm_assembly_6/urdf/arm_assembly_6.urdf (robot description, URDF)
Before this commit: robot arm_assembly_6, 7 links, 6 joints
Links:
- added link dummy_link
Joints:
- added joint dummy_joint: type fixed, parent dummy_link, child base_link
- joint joint1: axis 0 0 -1 -> 0 0 1
- joint joint2: axis 0 0 -1 -> 0 0 1; limit lower=0 upper=3.1415 effort=0 velocity=0 -> lower=-1.5708 upper=1.5708 effort=0 velocity=0
- joint joint3: axis 0 0 -1 -> 0 0 1; limit lower=0 upper=3.1415 effort=0 velocity=0 -> lower=-1.5708 upper=1.5708 effort=0 velocity=0
- joint joint4: axis 0 -0.00012785 -1 -> 0 0 1; limit lower=0 upper=3.1415 effort=0 velocity=0 -> lower=-1.5708 upper=1.5708 effort=0 velocity=0
- joint joint5: axis -0.00012785 0 -1 -> 0 0 1; limit lower=0 upper=3.1415 effort=0 velocity=0 -> lower=-1.5708 upper=1.5708 effort=0 velocity=0
- joint joint6: axis 0 -9.1989E-05 -1 -> 0 0 1; limit lower=0 upper=3.1415 effort=0 velocity=0 -> lower=-1.5708 upper=1.5708 effort=0 velocity=0
