Commit message: AISR description added

File: xarm_ws/src/aisr/urdf/aisr(复件).urdf (robot description, URDF)
Before this commit: robot aisr_description, 19 links, 18 joints
Links:
- removed link dummy_link
- added link world
- link Black_Link1: geometry collision mesh filename=package://aisr/meshes/Black_Link1.STL; visual mesh filename=package://aisr/meshes/Black_Link1.STL
- link Black_Link2: geometry collision mesh filename=package://aisr/meshes/Black_Link2.STL; visual mesh filename=package://aisr/meshes/Black_Link2.STL
- link Black_Link4: geometry collision mesh filename=package://aisr/meshes/Black_Link4.STL; visual mesh filename=package://aisr/meshes/Black_Link4.STL
- link Black_Link5: geometry collision mesh filename=package://aisr/meshes/Black_Link5.STL; visual mesh filename=package://aisr/meshes/Black_Link5.STL
- link Black_Link6: geometry collision mesh filename=package://aisr/meshes/Black_Link6.STL; visual mesh filename=package://aisr/meshes/Black_Link6.STL
- link Black_Link7: geometry collision mesh filename=package://aisr/meshes/Black_Link7.STL; visual mesh filename=package://aisr/meshes/Black_Link7.STL
- link Neck_Link1: geometry collision mesh filename=package://aisr/meshes/Neck_Link1.STL; visual mesh filename=package://aisr/meshes/Neck_Link1.STL
- link Neck_Link2: geometry collision mesh filename=package://aisr/meshes/Neck_Link2.STL; visual mesh filename=package://aisr/meshes/Neck_Link2.STL
- link Waist_Link1: geometry collision mesh filename=package://aisr/meshes/Waist_Link1.STL; visual mesh filename=package://aisr/meshes/Waist_Link1.STL
- link Waist_Link2: geometry collision mesh filename=package://aisr/meshes/Waist_Link2.STL; visual mesh filename=package://aisr/meshes/Waist_Link2.STL
- link Waist_Link3: geometry collision mesh filename=package://aisr/meshes/Waist_Link3.STL; visual mesh filename=package://aisr/meshes/Waist_Link3.STL
- link White_Link1: geometry collision mesh filename=package://aisr/meshes/White_Link1.STL; visual mesh filename=package://aisr/meshes/White_Link1.STL
- link White_Link2: geometry collision mesh filename=package://aisr/meshes/White_Link2.STL; visual mesh filename=package://aisr/meshes/White_Link2.STL
- link White_Link3: geometry collision mesh filename=package://aisr/meshes/White_Link3.STL; visual mesh filename=package://aisr/meshes/White_Link3.STL
- link White_Link4: geometry collision mesh filename=package://aisr/meshes/White_Link4.STL; visual mesh filename=package://aisr/meshes/White_Link4.STL
- link White_Link5: geometry collision mesh filename=package://aisr/meshes/White_Link5.STL; visual mesh filename=package://aisr/meshes/White_Link5.STL
- link base_link: geometry collision mesh filename=package://aisr/meshes/base_link.STL; visual mesh filename=package://aisr/meshes/base_link.STL
- link black_Link3: geometry collision mesh filename=package://aisr/meshes/black_Link3.STL; visual mesh filename=package://aisr/meshes/black_Link3.STL
Joints:
- removed joint black1
- removed joint black2
- removed joint black3
- removed joint black4
- removed joint black5
- removed joint black6
- removed joint black7
- removed joint dummy_joint
- removed joint neck1
- removed joint neck2
- removed joint waist1
- removed joint waist2
- removed joint waist3
- removed joint white1
- removed joint white2
- removed joint white3
- removed joint white4
- removed joint white5
- added joint black1_joint: type revolute, parent Waist_Link3, child Black_Link1, origin xyz=-0.13313 -0.14666 -0.0002 rpy=-1.5708 0 -1.309, axis 0 0 -1, limit lower=-2.0 upper=0.0 effort=100.0 velocity=1.0
- added joint black2_joint: type revolute, parent Black_Link1, child Black_Link2, origin xyz=0 0 -0.1165 rpy=-1.5708 -1.309 0, axis 0 0 -1, limit lower=0.0 upper=1.5 effort=100.0 velocity=1.0
- added joint black3_joint: type revolute, parent Black_Link2, child black_Link3, origin xyz=0 -0.11415 -0.0002 rpy=-1.5708 0 0, axis 0 0 -1, limit lower=-1.5 upper=1.5 effort=100.0 velocity=1.0
- added joint black4_joint: type revolute, parent black_Link3, child Black_Link4, origin xyz=0 0 -0.1482 rpy=1.5708 0 1.5708, axis 0 0 1, limit lower=0.0 upper=2.0 effort=100.0 velocity=1.0
- added joint black5_joint: type revolute, parent Black_Link4, child Black_Link5, origin xyz=0 -0.10775 0 rpy=-1.5708 -1.5708 0, axis 0 0 -1, limit lower=-1.5 upper=1.5 effort=100.0 velocity=1.0
- added joint black6_joint: type revolute, parent Black_Link5, child Black_Link6, origin xyz=0 0 -0.0481 rpy=1.5708 0 0, axis 0 0 1, limit lower=-1.5 upper=1.5 effort=100.0 velocity=1.0
- added joint black7_joint: type revolute, parent Black_Link6, child Black_Link7, origin xyz=0 -0.078 0 rpy=0 1.5708 0, axis 0 0 -1, limit lower=-1.5 upper=1.5 effort=100.0 velocity=1.0
- added joint fixed: type fixed, parent world, child base_link
- added joint neck1_joint: type revolute, parent Waist_Link3, child Neck_Link1, origin xyz=0.0005 -0.22275 -0.0002 rpy=1.5708 0 0, axis 0 0 -1, limit lower=-0.2 upper=0.2 effort=100.0 velocity=1.0
- added joint neck2_joint: type revolute, parent Neck_Link1, child Neck_Link2, origin xyz=0.0002 0 0.0415 rpy=1.5708 0 1.5708, axis 0 0 -1, limit lower=-0.2 upper=0.2 effort=100.0 velocity=1.0
- added joint waist1_joint: type revolute, parent base_link, child Waist_Link1, origin xyz=0 0 0.5625 rpy=0 0 -1.5707963267949, axis 0 0 -1, limit lower=-0.2 upper=0.2 effort=100.0 velocity=1.0
- added joint waist2_joint: type revolute, parent Waist_Link1, child Waist_Link2, origin xyz=0 0 0.0685 rpy=-1.5708 0 1.5708, axis 0 0 -1, limit lower=-0.01 upper=0.01 effort=100.0 velocity=1.0
- added joint waist3_joint: type revolute, parent Waist_Link2, child Waist_Link3, origin xyz=0 -0.105 0.0007 rpy=0 1.5708 0, axis 0 0 1, limit lower=-0.01 upper=0.01 effort=100.0 velocity=1.0
- added joint white1_joint: type revolute, parent Waist_Link3, child White_Link1, origin xyz=0.20962 -0.16689 -0.0002 rpy=1.5708 0 1.309, axis 0 0 1, limit lower=0.0 upper=2.0 effort=100.0 velocity=1.0
- added joint white2_joint: type revolute, parent White_Link1, child White_Link2, origin xyz=0 0 0.055 rpy=1.5708 -1.309 0, axis 0 0 1, limit lower=0.0 upper=1.5 effort=100.0 velocity=1.0
- added joint white3_joint: type revolute, parent White_Link2, child White_Link3, origin xyz=0 -0.08 0.0045 rpy=-1.5708 0 0, axis 0 0 -1, limit lower=-1.5 upper=1.5 effort=100.0 velocity=1.0
- added joint white4_joint: type revolute, parent White_Link3, child White_Link4, origin xyz=0 0 -0.163 rpy=1.5708 0 1.5708, axis 0 0 1, limit lower=0.0 upper=2.0 effort=100.0 velocity=1.0
- added joint white5_joint: type revolute, parent White_Link4, child White_Link5, origin xyz=0 -0.06 0 rpy=-1.5708 -1.5708 0, axis 0 0 -1, limit lower=-1.5 upper=1.5 effort=100.0 velocity=1.0
