Commit message: AISR updated

File: xarm_ws/src/aisr/urdf/aisr.urdf (robot description, URDF)
Before this commit: robot aisr, 19 links, 18 joints
Links:
- removed link world
- added link dummy_link
Joints:
- removed joint fixed
- added joint dummy_joint: type fixed, parent dummy_link, child base_link

Commit message: aisr model updated

File: xarm_ws/src/aisr/urdf/aisr.urdf (robot description, URDF)
Before this commit: robot aisr, 19 links, 18 joints
Links:
- added link Link1, mass 0.00330620599604871; collision mesh filename=package://aisr/meshes/r_hand/Link1.STL; visual mesh filename=package://aisr/meshes/r_hand/Link1.STL
- added link Link11, mass 0.00453366822308025; collision mesh filename=package://aisr/meshes/r_hand/Link11.STL; visual mesh filename=package://aisr/meshes/r_hand/Link11.STL
- added link Link111, mass 0.22621959250221; collision mesh filename=package://aisr/meshes/r_hand/Link111.STL; visual mesh filename=package://aisr/meshes/r_hand/Link111.STL
- added link Link2, mass 0.00330621565435093; collision mesh filename=package://aisr/meshes/r_hand/Link2.STL; visual mesh filename=package://aisr/meshes/r_hand/Link2.STL
- added link Link22, mass 0.00453367017295165; collision mesh filename=package://aisr/meshes/r_hand/Link22.STL; visual mesh filename=package://aisr/meshes/r_hand/Link22.STL
- added link Link3, mass 0.0033061482917439; collision mesh filename=package://aisr/meshes/r_hand/Link3.STL; visual mesh filename=package://aisr/meshes/r_hand/Link3.STL
- added link Link33, mass 0.00453366652527048; collision mesh filename=package://aisr/meshes/r_hand/Link33.STL; visual mesh filename=package://aisr/meshes/r_hand/Link33.STL
- added link Link4, mass 0.00330620800050046; collision mesh filename=package://aisr/meshes/r_hand/Link4.STL; visual mesh filename=package://aisr/meshes/r_hand/Link4.STL
- added link Link44, mass 0.00356886192445218; collision mesh filename=package://aisr/meshes/r_hand/Link44.STL; visual mesh filename=package://aisr/meshes/r_hand/Link44.STL
- added link Link5, mass 0.00487390663164139; collision mesh filename=package://aisr/meshes/r_hand/Link5.STL; visual mesh filename=package://aisr/meshes/r_hand/Link5.STL
- added link Link51, mass 0.00652729219675812; collision mesh filename=package://aisr/meshes/r_hand/Link51.STL; visual mesh filename=package://aisr/meshes/r_hand/Link51.STL
- added link Link52, mass 0.0022695308360543; collision mesh filename=package://aisr/meshes/r_hand/Link52.STL; visual mesh filename=package://aisr/meshes/r_hand/Link52.STL
- added link Link53, mass 0.00330869751403717; collision mesh filename=package://aisr/meshes/r_hand/Link53.STL; visual mesh filename=package://aisr/meshes/r_hand/Link53.STL
Joints:
- added joint Link1: type fixed, parent Link111, child Link1, origin xyz=0.08225 -0.0077547 -0.0040172 rpy=5.2178E-10 -6.245E-17 -0.14966, axis 0 0 1, limit lower=-1.6 upper=0 effort=1 velocity=1
- added joint Link11: type fixed, parent Link1, child Link11, origin xyz=0.032132 0 0 rpy=-5.086E-10 -1.1653E-10 -0.22524, axis 0 0 1, limit lower=-1.7 upper=0 effort=1 velocity=1
- added joint Link2: type fixed, parent Link111, child Link2, origin xyz=0.081939 -0.0077547 0.015305 rpy=0.0056158 -0.034452 -0.16161, axis 0 0 1, limit lower=-1.6 upper=0 effort=1 velocity=1
- added joint Link22: type fixed, parent Link2, child Link22, origin xyz=0.032132 0 0 rpy=-5.0853E-10 -1.1686E-10 -0.22588, axis 0 0 1, limit lower=-1.7 upper=0 effort=1 velocity=1
- added joint Link3: type fixed, parent Link111, child Link3, origin xyz=0.080765 -0.0077547 0.034505 rpy=0.010408 -0.086645 -0.11971, axis 0 0 1, limit lower=-1.6 upper=0 effort=1 velocity=1
- added joint Link33: type fixed, parent Link3, child Link33, origin xyz=0.032132 0 0 rpy=-5.0314E-10 -1.3824E-10 -0.26815, axis 0 0 1, limit lower=-1.7 upper=0 effort=1 velocity=1
- added joint Link4: type fixed, parent Link111, child Link4, origin xyz=0.078587 -0.0077547 0.053617 rpy=0.022524 -0.13781 -0.16255, axis 0 0 1, limit lower=-1.6 upper=0 effort=1 velocity=1
- added joint Link44: type fixed, parent Link4, child Link44, origin xyz=0.032132 0 0 rpy=-5.0686E-10 -1.2389E-10 -0.23972, axis 0 0 1, limit lower=-1.7 upper=0 effort=1 velocity=1
- added joint Link5: type fixed, parent Link111, child Link5, origin xyz=0.0089225 -0.022949 -0.00699 rpy=0.092365 1.1827 -1.4853, axis 0 1 0, limit lower=-1 upper=0.3 effort=1 velocity=1
- added joint Link51: type fixed, parent Link5, child Link51, origin xyz=0.0065 -0.0035 0.00425 rpy=3.1416 -5.2736E-16 0.96726, axis 0 0 -1, limit lower=0 upper=0.4 effort=1 velocity=1
- added joint Link52: type fixed, parent Link51, child Link52, origin xyz=0.056001 0 0 rpy=0 -1.3878E-16 2.9661, axis 0 0 1, limit lower=-0.4 upper=0 effort=1 velocity=1
- added joint Link53: type fixed, parent Link52, child Link53, origin xyz=-0.022653 0 0 rpy=1.7291 -1.5708 0, axis 1 0 0, limit lower=-1 upper=0 effort=1 velocity=1
- added joint white_hand: type revolute, parent White_Link5, child Link111, origin xyz=0 0 -0.275 rpy=-1.57 1.57 3.14, axis -1 0 0, limit lower=-3.14 upper=3.14 effort=100.0 velocity=1.0

Commit message: xarm_ws updated, trying to use xarm API for controlling

File: xarm_ws/src/aisr/urdf/aisr.urdf (robot description, URDF)
Before this commit: robot aisr, 32 links, 31 joints
Links:
- removed link White_Link1
- removed link White_Link2
- removed link White_Link3
- removed link White_Link4
- removed link White_Link5
- added link link1, mass 0.46221855499898; collision mesh filename=package://aisr/meshes/White_Link1.STL; visual mesh filename=package://aisr/meshes/White_Link1.STL
- added link link2, mass 0.103619832607522; collision mesh filename=package://aisr/meshes/White_Link2.STL; visual mesh filename=package://aisr/meshes/White_Link2.STL
- added link link3, mass 0.600118848773854; collision mesh filename=package://aisr/meshes/White_Link3.STL; visual mesh filename=package://aisr/meshes/White_Link3.STL
- added link link4, mass 0.0620799654815404; collision mesh filename=package://aisr/meshes/White_Link4.STL; visual mesh filename=package://aisr/meshes/White_Link4.STL
- added link link5, mass 0.439408367700066; collision mesh filename=package://aisr/meshes/White_Link5.STL; visual mesh filename=package://aisr/meshes/White_Link5.STL
- added link link6
- added link link7
- added link link_eef
Joints:
- removed joint white1_joint
- removed joint white2_joint
- removed joint white3_joint
- removed joint white4_joint
- removed joint white5_joint
- added joint joint1: type revolute, parent Waist_Link3, child link1, origin xyz=0.20962 -0.16689 -0.0002 rpy=1.5708 0 1.309, axis 0 0 1, limit lower=0.0 upper=2.0 effort=100.0 velocity=1.0
- added joint joint2: type revolute, parent link1, child link2, origin xyz=0 0 0.055 rpy=1.5708 -1.5708 0, axis 0 0 1, limit lower=0.0 upper=1.5 effort=100.0 velocity=1.0
- added joint joint3: type revolute, parent link2, child link3, origin xyz=0 -0.08 0.0045 rpy=-1.5708 0 0, axis 0 0 -1, limit lower=-1.5 upper=1.5 effort=100.0 velocity=1.0
- added joint joint4: type revolute, parent link3, child link4, origin xyz=0 0 -0.163 rpy=1.5708 0 1.5708, axis 0 0 1, limit lower=0.0 upper=2.0 effort=100.0 velocity=1.0
- added joint joint5: type revolute, parent link4, child link5, origin xyz=0 -0.06 0 rpy=-1.5708 -1.5708 0, axis 0 0 -1, limit lower=-1.5 upper=1.5 effort=100.0 velocity=1.0
- added joint joint6: type fixed, parent link5, child link6, origin xyz=0 0 0 rpy=0 0 0
- added joint joint7: type fixed, parent link6, child link7, origin xyz=0 0 -0.23 rpy=0 0 0
- added joint joint_eef: type fixed, parent link7, child link_eef, origin xyz=0 0 0 rpy=0 0 0
- joint white_hand: origin xyz=0 0 -0.275 rpy=-1.57 1.57 3.14 -> xyz=0 0 -0.045 rpy=-1.57 1.57 3.14; parent White_Link5 -> link_eef

Commit message: AISR drawing a circle with moveit completed

File: xarm_ws/src/aisr/urdf/aisr.urdf (robot description, URDF)
Before this commit: robot aisr, 35 links, 34 joints
Joints:
- joint joint7: origin xyz=0 0 -0.23 rpy=0 0 0 -> xyz=0 -0.12000024 -0.325247 rpy=0 0 0
- joint joint_eef: origin xyz=0 0 0 rpy=0 0 0 -> xyz=0 0.12000024 0.095247 rpy=0 0 0

Commit message: Writing Chinese character '福' and drawing circle with AISR's white arm completed

File: xarm_ws/src/aisr/urdf/aisr.urdf (robot description, URDF)
Before this commit: robot aisr, 35 links, 34 joints
Joints:
- joint Link1: limit lower=-1.6 upper=0 effort=1 velocity=1 -> lower=-1.6 upper=0 effort=1 velocity=100
- joint Link11: limit lower=-1.7 upper=0 effort=1 velocity=1 -> lower=-1.7 upper=0 effort=1 velocity=100
- joint Link2: limit lower=-1.6 upper=0 effort=1 velocity=1 -> lower=-1.6 upper=0 effort=1 velocity=100
- joint Link22: limit lower=-1.7 upper=0 effort=1 velocity=1 -> lower=-1.7 upper=0 effort=1 velocity=100
- joint Link3: limit lower=-1.6 upper=0 effort=1 velocity=1 -> lower=-1.6 upper=0 effort=1 velocity=100
- joint Link33: limit lower=-1.7 upper=0 effort=1 velocity=1 -> lower=-1.7 upper=0 effort=1 velocity=100
- joint Link4: limit lower=-1.6 upper=0 effort=1 velocity=1 -> lower=-1.6 upper=0 effort=1 velocity=100
- joint Link44: limit lower=-1.7 upper=0 effort=1 velocity=1 -> lower=-1.7 upper=0 effort=1 velocity=100
- joint Link5: limit lower=-1 upper=0.3 effort=1 velocity=1 -> lower=-1 upper=0.3 effort=1 velocity=100
- joint Link51: limit lower=0 upper=0.4 effort=1 velocity=1 -> lower=0 upper=0.4 effort=1 velocity=100
- joint Link52: limit lower=-0.4 upper=0 effort=1 velocity=1 -> lower=-0.4 upper=0 effort=1 velocity=100
- joint Link53: limit lower=-1 upper=0 effort=1 velocity=1 -> lower=-1 upper=0 effort=1 velocity=100
- joint black1_joint: limit lower=-2.0 upper=0.0 effort=100.0 velocity=1.0 -> lower=-2.0 upper=0.0 effort=100.0 velocity=100.0
- joint black2_joint: limit lower=0.0 upper=1.5 effort=100.0 velocity=1.0 -> lower=0.0 upper=1.5 effort=100.0 velocity=100.0
- joint black3_joint: limit lower=-1.5 upper=1.5 effort=100.0 velocity=1.0 -> lower=-1.5 upper=1.5 effort=100.0 velocity=100.0
- joint black4_joint: limit lower=0.0 upper=2.0 effort=100.0 velocity=1.0 -> lower=0.0 upper=2.0 effort=100.0 velocity=100.0
- joint black5_joint: limit lower=-1.5 upper=1.5 effort=100.0 velocity=1.0 -> lower=-1.5 upper=1.5 effort=100.0 velocity=100.0
- joint black6_joint: limit lower=-1.5 upper=1.5 effort=100.0 velocity=1.0 -> lower=-1.5 upper=1.5 effort=100.0 velocity=100.0
- joint black7_joint: limit lower=-1.5 upper=1.5 effort=100.0 velocity=1.0 -> lower=-1.5 upper=1.5 effort=100.0 velocity=100.0
- joint joint1: limit lower=0.0 upper=2.0 effort=100.0 velocity=1.0 -> lower=0.0 upper=2.0 effort=100.0 velocity=100.0
- joint joint2: limit lower=0.0 upper=1.5 effort=100.0 velocity=1.0 -> lower=0.0 upper=1.5 effort=100.0 velocity=100.0
- joint joint3: limit lower=-1.5 upper=1.5 effort=100.0 velocity=1.0 -> lower=-1.5 upper=1.5 effort=100.0 velocity=100.0
- joint joint4: limit lower=0.0 upper=2.0 effort=100.0 velocity=1.0 -> lower=0.0 upper=2.0 effort=100.0 velocity=100.0
- joint joint5: limit lower=-1.5 upper=1.5 effort=100.0 velocity=1.0 -> lower=-1.5 upper=1.5 effort=100.0 velocity=100.0
- joint neck1_joint: limit lower=-1.5 upper=1.5 effort=100.0 velocity=1.0 -> lower=-1.5 upper=1.5 effort=100.0 velocity=100.0
- joint neck2_joint: limit lower=-0.5 upper=0.5 effort=100.0 velocity=1.0 -> lower=-0.5 upper=0.5 effort=100.0 velocity=100.0
- joint waist1_joint: limit lower=-1.0 upper=1.0 effort=100.0 velocity=1.0 -> lower=-1.0 upper=1.0 effort=100.0 velocity=100.0
- joint waist2_joint: limit lower=-0.5 upper=0.5 effort=100.0 velocity=1.0 -> lower=-0.5 upper=0.5 effort=100.0 velocity=100.0
- joint waist3_joint: limit lower=-0.5 upper=0.5 effort=100.0 velocity=1.0 -> lower=-0.5 upper=0.5 effort=100.0 velocity=100.0
- joint white_hand: limit lower=-3.14 upper=3.14 effort=100.0 velocity=1.0 -> lower=-3.14 upper=3.14 effort=100.0 velocity=100.0
